Commit message: Presentation material

File: urdf/scancontrol.xacro (robot description, xacro)
@@ -46,12 +46,12 @@
                         <samples>1024</samples>
                         <resolution>1</resolution>
-                        <min_angle>-${M_PI/8}</min_angle>
-                        <max_angle>${M_PI/8}</max_angle>
+                        <min_angle>-${M_PI/16}</min_angle>
+                        <max_angle>${M_PI/16}</max_angle>
                     </horizontal>
                 </scan>
                 <range>
-                    <min>0.1</min>
+                    <min>0.0</min>
                     <max>0.500</max>
-                    <resolution>0.01</resolution>
+                    <resolution>0.001</resolution>
                 </range>
             </ray>

File: urdf/welding_sensor.xacro (robot description, xacro)
@@ -2,4 +2,5 @@
 <robot xmlns:xacro="http://www.ros.org/wiki/xacro" name="welding_sensor">
   <xacro:macro name="welding_sensor" params="parent">
+    <xacro:property name="M_PI" value="3.1415926535897931" />
     <!-- ======================= Links ======================= -->
     <link name="Weldingsensor">
@@ -17,14 +18,14 @@
       </collision>
       <inertial>
-        <origin xyz="0.0 -0.0688 -0.0428" rpy="0.0 0.0 0.0"/>
-        <mass value="0.8" />
-        <inertia ixx="0.0029" ixy="-0.0000" ixz="-0.0000"
-                 iyy="0.0009" iyz="0.0001"
-                 izz="0.0030"/>
+        <origin xyz="0.0 0 0" rpy="0.0 0.0 0.0"/>
+        <mass value="0.00001" />
+        <inertia ixx="0.000001" ixy="0.0000" ixz="0.0000"
+                 iyy="0.000001" iyz="0.0000"
+                 izz="0.000001"/>
       </inertial>
     </link>
     <link name="laser_beam">
       <visual>
-        <origin xyz="0 -0.013 0" rpy="-1.5708 0 0"/>
+        <origin xyz="-0.013 0 0" rpy="0 -1.5708 0"/>
         <geometry>
           <cylinder radius="0.01" length="0.01"/>
@@ -32,5 +33,5 @@
       </visual>
       <collision>
-        <origin xyz="0 -0.013 0" rpy="-1.5708 0 0"/>
+        <origin xyz="-0.013 0 0" rpy="0 -1.5708 0"/>
         <geometry>
           <cylinder radius="0.01" length="0.01"/>
@@ -48,8 +49,8 @@
       <parent link="${parent}"/>
       <child  link="Weldingsensor"/>
-      <origin xyz="-0.013 0.065 0.119" rpy="1.5708 0 0"/>
+      <origin xyz="0 0 0" rpy="1.5708 0 0"/>
     </joint>
     <joint name="laser_emitter" type="fixed">
-      <origin xyz="0 0 0" rpy="1.5708 0 0"/>
+      <origin xyz="0 0 0" rpy="-1.5708 -1.5708 0"/>
       <parent link="Weldingsensor"/>
       <child link="laser_beam"/>
@@ -69,11 +70,11 @@
               <samples>640</samples>
               <resolution>1</resolution>
-              <min_angle>1.3963</min_angle>
-              <max_angle>1.7453</max_angle>
+              <min_angle>-${M_PI/12}</min_angle>
+              <max_angle>${M_PI/12}</max_angle>
             </horizontal>
           </scan>
           <range>
-            <min>0.3</min>
-            <max>.6</max>
+            <min>0.2</min>
+            <max>.5</max>
             <resolution>0.01</resolution>
           </range>
